Commit message: new changes

File: src/my_bot/description/robot_core.xacro (robot description, xacro)
@@ -6,5 +6,5 @@
     <xacro:property name="chassis_height" value="0.1" />
     <xacro:property name="chassis_mass" value="1.0" />
-    <xacro:property name="wheel_radius" value="0.033" />
+    <xacro:property name="wheel_radius" value="0.027" />
     <xacro:property name="wheel_thickness" value="0.026" />
     <xacro:property name="wheel_mass" value="0.05" />
