Commit message: new_worlds added

File: src/my_bot/description/robot.urdf.xacro (robot description, xacro)
@@ -5,5 +5,5 @@
     <xacro:include filename="robot_core.xacro" />
     <xacro:if value="$(arg use_ros2_control)">
-        <xacro:include filename="ros2_control.xacro" />
+        <xacro:include filename="ros2_control2.xacro" />
     </xacro:if>
     <xacro:unless value="$(arg use_ros2_control)">
@@ -11,5 +11,5 @@
     </xacro:unless>
     <xacro:include filename="lidar.xacro" />
-    <!-- <xacro:include filename="gazebo_control.xacro" /> -->
+    <xacro:include filename="gazebo_control.xacro" />
     <!-- <xacro:include filename="camera.xacro" /> -->
     <!-- <xacro:include filename="depth_camera.xacro" /> -->

File: src/my_bot/description/robot_core.xacro (robot description, xacro)
@@ -6,5 +6,5 @@
     <xacro:property name="chassis_height" value="0.1" />
     <xacro:property name="chassis_mass" value="1.0" />
-    <xacro:property name="wheel_radius" value="0.027" />
+    <xacro:property name="wheel_radius" value="0.03" />
     <xacro:property name="wheel_thickness" value="0.026" />
     <xacro:property name="wheel_mass" value="0.05" />
